File: extras/transmitter_SI5351_Arduinol.sch (EAGLE design)
At the start: 16 parts, among them M2 ARDUINO-PRO-MINI-3.3V#APC, Q1-2N3904 200mA/40V, Q2-2N3904 200mA/40V, U1 SI5351B-B-GM, X1 12MHz

Commit message: PU2CLR Sortwave Transmitter
Parts:
- removed X1: 12MHz, adafruit:CRYSTAL68SMX
- added C5: 10nF, rcl:CXXC10B6
Connections:
- new net N$2: C5.1, Q2-2N3904.B, R1.1
- net N$3: no longer X1.2
- net N$9: now also C5.2; no longer Q2-2N3904.B, R1.1, X1.1
Changed lines of the file:
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@@
 <part name="Q2-2N3904" library="SparkFun-DiscreteSemi" library_urn="urn:adsk.eagle:library:514" deviceset="TRANS_NPN" device="-2N3904" package3d_urn="urn:adsk.eagle:package:38450/1" value="200mA/40V"/>
 <part name="C1" library="rcl" library_urn="urn:adsk.eagle:library:334" deviceset="CX" device="XC10B6" package3d_urn="urn:adsk.eagle:package:23700/1" value="47pF"/>
-<part name="X1" library="adafruit" library_urn="urn:adsk.eagle:library:420" deviceset="CRYSTAL" device="68SMX" package3d_urn="urn:adsk.eagle:package:6240918/1" value="12MHz"/>
 <part name="R1" library="Resistor" library_urn="urn:adsk.eagle:library:16378527" deviceset="R-US" device="AXIAL-7.2MM-PITCH" package3d_urn="urn:adsk.eagle:package:16378561/2" technology="_" value="100K"/>
 <part name="R2" library="Resistor" library_urn="urn:adsk.eagle:library:16378527" deviceset="R-US" device="AXIAL-7.2MM-PITCH" package3d_urn="urn:adsk.eagle:package:16378561/2" technology="_" value="1K"/>
@@
 </part>
 <part name="GND2" library="supply1" library_urn="urn:adsk.eagle:library:371" deviceset="GND" device=""/>
+<part name="C5" library="rcl" library_urn="urn:adsk.eagle:library:334" deviceset="CX" device="XC10B6" package3d_urn="urn:adsk.eagle:package:23700/1" value="10nF"/>
 </parts>
 <sheets>
@@
 <attribute name="VALUE" x="118.364" y="46.101" size="1.778" layer="96"/>
 </instance>
-<instance part="X1" gate="G$1" x="76.2" y="55.88" smashed="yes" rot="R90">
-<attribute name="NAME" x="72.644" y="53.34" size="1.778" layer="95" rot="R90"/>
-<attribute name="VALUE" x="73.66" y="43.18" size="1.778" layer="96" rot="R90"/>
-</instance>
 <instance part="R1" gate="G$1" x="81.28" y="55.88" smashed="yes" rot="R90">
 <attribute name="NAME" x="88.6714" y="55.88" size="1.778" layer="95" rot="R90" align="center"/>
@@
 <instance part="GND2" gate="1" x="73.66" y="-66.04" smashed="yes">
 <attribute name="VALUE" x="71.12" y="-68.58" size="1.778" layer="96"/>
+</instance>
+<instance part="C5" gate="G$1" x="81.28" y="22.86" smashed="yes">
+<attribute name="NAME" x="77.724" y="25.781" size="1.778" layer="95"/>
+<attribute name="VALUE" x="85.344" y="23.241" size="1.778" layer="96"/>
 </instance>
 </instances>
@@
 <pinref part="R2" gate="G$1" pin="2"/>
 <wire x1="63.5" y1="50.8" x2="63.5" y2="60.96" width="0.1524" layer="91"/>
-<pinref part="X1" gate="G$1" pin="2"/>
-<wire x1="76.2" y1="58.42" x2="76.2" y2="60.96" width="0.1524" layer="91"/>
 <pinref part="R1" gate="G$1" pin="2"/>
-<wire x1="76.2" y1="60.96" x2="81.28" y2="60.96" width="0.1524" layer="91"/>
 <wire x1="81.28" y1="60.96" x2="91.44" y2="60.96" width="0.1524" layer="91"/>
 <junction x="81.28" y="60.96"/>
@@
 <wire x1="91.44" y1="60.96" x2="91.44" y2="50.8" width="0.1524" layer="91"/>
 <junction x="91.44" y="50.8"/>
-<wire x1="63.5" y1="60.96" x2="76.2" y2="60.96" width="0.1524" layer="91"/>
-<junction x="76.2" y="60.96"/>
+<wire x1="63.5" y1="60.96" x2="81.28" y2="60.96" width="0.1524" layer="91"/>
 </segment>
 </net>
 <net name="N$9" class="0">
 <segment>
-<pinref part="X1" gate="G$1" pin="1"/>
-<wire x1="76.2" y1="53.34" x2="76.2" y2="45.72" width="0.1524" layer="91"/>
-<pinref part="Q2-2N3904" gate="G$1" pin="B"/>
-<wire x1="76.2" y1="45.72" x2="81.28" y2="45.72" width="0.1524" layer="91"/>
-<pinref part="R1" gate="G$1" pin="1"/>
-<wire x1="81.28" y1="45.72" x2="86.36" y2="45.72" width="0.1524" layer="91"/>
-<wire x1="81.28" y1="50.8" x2="81.28" y2="45.72" width="0.1524" layer="91"/>
-<junction x="81.28" y="45.72"/>
 <pinref part="U1" gate="G$1" pin="CLK0"/>
 <wire x1="119.38" y1="-27.94" x2="134.62" y2="-27.94" width="0.1524" layer="91"/>
 <wire x1="134.62" y1="-27.94" x2="134.62" y2="17.78" width="0.1524" layer="91"/>
 <wire x1="134.62" y1="17.78" x2="81.28" y2="17.78" width="0.1524" layer="91"/>
-<wire x1="81.28" y1="17.78" x2="81.28" y2="45.72" width="0.1524" layer="91"/>
-</segment>
-</net>
+<pinref part="C5" gate="G$1" pin="2"/>
+</segment>
+</net>
+<net name="N$2" class="0">
+<segment>
+<pinref part="Q2-2N3904" gate="G$1" pin="B"/>
+<wire x1="81.28" y1="45.72" x2="86.36" y2="45.72" width="0.1524" layer="91"/>
+<pinref part="R1" gate="G$1" pin="1"/>
+<wire x1="81.28" y1="50.8" x2="81.28" y2="45.72" width="0.1524" layer="91"/>
+<junction x="81.28" y="45.72"/>
+<pinref part="C5" gate="G$1" pin="1"/>
+<wire x1="81.28" y1="25.4" x2="81.28" y2="45.72" width="0.1524" layer="91"/>
+</segment>
+</net>

Commit message: Shortwave receiver tester
Parts:
- removed INPUT: POWER_JACKPTH_SMD_COMBO, SparkFun-Connectors:POWER_JACKPTH_SMD_COMBO
- added AUDIO_INPUT: POWER_JACKPTH_SMD_COMBO, SparkFun-Connectors:POWER_JACKPTH_SMD_COMBO
- added S1: (no value), SparkFun-Switches:ENCODER
- added SW1: (no value), adafruit:SWITCH_PUSHBUTTONC&K_KSS
- added U$2: DISPLAY-OLED-128X64-I2C, diy-modules:DISPLAY-OLED-128X64-I2C
Connections:
- new net N$10: M2.D2, S1.A
- new net N$11: M2.D3, S1.B
- new net N$12: M2.D4, SW1.P$2
- net GND: now also AUDIO_INPUT.PWR, S1.C, SW1.P$1, U$2.GND; no longer INPUT.PWR
- net N$1: now also AUDIO_INPUT.GND; no longer INPUT.GND
- net N$7: now also U$2.SDA
- net N$8: now also U$2.SCL
- net VCC: now also U$2.VCC
Other:
- moved on the sheet: C3
Changed lines of the file:
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@@
 </part>
 <part name="C4" library="SparkFun-Capacitors" library_urn="urn:adsk.eagle:library:510" deviceset="100UF-POLAR" device="-10X10.5-63V-20%" package3d_urn="urn:adsk.eagle:package:37417/1" value="100uF"/>
-<part name="INPUT" library="SparkFun-Connectors" library_urn="urn:adsk.eagle:library:513" deviceset="POWER_JACK" device="PTH_SMD_COMBO" package3d_urn="urn:adsk.eagle:package:38223/1"/>
+<part name="AUDIO_INPUT" library="SparkFun-Connectors" library_urn="urn:adsk.eagle:library:513" deviceset="POWER_JACK" device="PTH_SMD_COMBO" package3d_urn="urn:adsk.eagle:package:38223/1"/>
 <part name="ANT1" library="discrete" library_urn="urn:adsk.eagle:library:211" deviceset="ANTENNA" device="" package3d_urn="urn:adsk.eagle:package:12928/1"/>
 <part name="SUPPLY2" library="supply2" library_urn="urn:adsk.eagle:library:372" deviceset="VCC" device="">
@@
 <part name="GND2" library="supply1" library_urn="urn:adsk.eagle:library:371" deviceset="GND" device=""/>
 <part name="C5" library="rcl" library_urn="urn:adsk.eagle:library:334" deviceset="CX" device="XC10B6" package3d_urn="urn:adsk.eagle:package:23700/1" value="10nF"/>
+<part name="S1" library="SparkFun-Switches" library_urn="urn:adsk.eagle:library:535" deviceset="ENCODER" device="" package3d_urn="urn:adsk.eagle:package:40145/1"/>
+<part name="SW1" library="adafruit" library_urn="urn:adsk.eagle:library:420" deviceset="SWITCH_PUSHBUTTON" device="C&amp;K_KSS" package3d_urn="urn:adsk.eagle:package:6240958/1"/>
+<part name="SUPPLY3" library="supply2" library_urn="urn:adsk.eagle:library:372" deviceset="VCC" device="">
+<attribute name="TR_VCC" value="3.3V"/>
+</part>
+<part name="U$2" library="diy-modules" deviceset="DISPLAY-OLED-128X64-I2C" device=""/>
+<part name="GND3" library="supply1" library_urn="urn:adsk.eagle:library:371" deviceset="GND" device=""/>
 </parts>
 <sheets>
@@
 <instances>
 <instance part="M2" gate="G$1" x="17.78" y="-33.02" smashed="yes">
-<attribute name="NAME" x="-5.08" y="-5.08" size="1.778" layer="95"/>
-<attribute name="VALUE" x="5.08" y="0" size="1.778" layer="96"/>
+<attribute name="VALUE" x="-5.08" y="-66.04" size="1.778" layer="96"/>
 </instance>
 <instance part="U1" gate="G$1" x="104.14" y="-33.02" smashed="yes">
@@
 <attribute name="VALUE" x="25.4" y="49.022" size="1.778" layer="96" rot="R180" align="center"/>
 </instance>
-<instance part="C3" gate="G$1" x="12.7" y="17.78" smashed="yes" rot="R90">
-<attribute name="NAME" x="19.939" y="16.764" size="1.778" layer="95" rot="R180"/>
-<attribute name="VALUE" x="22.479" y="14.224" size="1.778" layer="96" rot="R180"/>
+<instance part="C3" gate="G$1" x="-12.7" y="63.5" smashed="yes" rot="R90">
+<attribute name="NAME" x="-5.461" y="62.484" size="1.778" layer="95" rot="R180"/>
+<attribute name="VALUE" x="-2.921" y="59.944" size="1.778" layer="96" rot="R180"/>
 </instance>
 <instance part="GND1" gate="1" x="68.58" y="27.94" smashed="yes">
@@
 <attribute name="VALUE" x="-4.064" y="44.069" size="1.778" layer="96" font="vector"/>
 </instance>
-<instance part="INPUT" gate="G$1" x="2.54" y="15.24" smashed="yes">
-<attribute name="NAME" x="-7.62" y="15.24" size="1.778" layer="95" font="vector"/>
+<instance part="AUDIO_INPUT" gate="G$1" x="-22.86" y="60.96" smashed="yes">
+<attribute name="NAME" x="-50.8" y="66.04" size="1.778" layer="95" font="vector"/>
 </instance>
 <instance part="ANT1" gate="A" x="116.84" y="66.04" smashed="yes">
@@
 <attribute name="NAME" x="77.724" y="25.781" size="1.778" layer="95"/>
 <attribute name="VALUE" x="85.344" y="23.241" size="1.778" layer="96"/>
+</instance>
+<instance part="S1" gate="G$1" x="-35.56" y="-33.02" smashed="yes">
+<attribute name="NAME" x="-40.64" y="-22.606" size="1.778" layer="95" font="vector"/>
+<attribute name="VALUE" x="-40.64" y="-43.434" size="1.778" layer="96" font="vector" align="top-left"/>
+</instance>
+<instance part="SW1" gate="G$1" x="-35.56" y="-53.34" smashed="yes">
+<attribute name="NAME" x="-38.1" y="-49.784" size="1.27" layer="95"/>
+<attribute name="VALUE" x="-38.1" y="-55.626" size="1.27" layer="96"/>
+</instance>
+<instance part="SUPPLY3" gate="G$1" x="-20.32" y="2.54" smashed="yes" rot="MR0">
+<attribute name="VALUE" x="-18.415" y="5.715" size="1.778" layer="96" rot="MR0" display="off"/>
+<attribute name="TR_VCC" x="-12.7" y="5.08" size="1.778" layer="96" rot="MR0"/>
+</instance>
+<instance part="U$2" gate="G$1" x="-53.34" y="-2.54" smashed="yes" rot="R270">
+<attribute name="VALUE" x="-38.1" y="17.78" size="1.778" layer="96" rot="R180"/>
+</instance>
+<instance part="GND3" gate="1" x="-20.32" y="76.2" smashed="yes" rot="R180">
+<attribute name="VALUE" x="-17.78" y="78.74" size="1.778" layer="96" rot="R180"/>
 </instance>
 </instances>
@@
 <wire x1="71.12" y1="-38.1" x2="71.12" y2="-15.24" width="0.1524" layer="91"/>
 <pinref part="M2" gate="G$1" pin="A4"/>
-<wire x1="71.12" y1="-15.24" x2="35.56" y2="-15.24" width="0.1524" layer="91"/>
+<wire x1="71.12" y1="-15.24" x2="40.64" y2="-15.24" width="0.1524" layer="91"/>
+<pinref part="U$2" gate="G$1" pin="SDA"/>
+<wire x1="40.64" y1="-15.24" x2="35.56" y2="-15.24" width="0.1524" layer="91"/>
+<wire x1="-33.02" y1="-5.08" x2="-5.08" y2="-5.08" width="0.1524" layer="91"/>
+<wire x1="-5.08" y1="-5.08" x2="-5.08" y2="5.08" width="0.1524" layer="91"/>
+<wire x1="-5.08" y1="5.08" x2="40.64" y2="5.08" width="0.1524" layer="91"/>
+<wire x1="40.64" y1="5.08" x2="40.64" y2="-15.24" width="0.1524" layer="91"/>
+<junction x="40.64" y="-15.24"/>
 </segment>
 </net>
@@
 <wire x1="73.66" y1="-35.56" x2="73.66" y2="-12.7" width="0.1524" layer="91"/>
 <pinref part="M2" gate="G$1" pin="A5"/>
-<wire x1="73.66" y1="-12.7" x2="35.56" y2="-12.7" width="0.1524" layer="91"/>
+<wire x1="73.66" y1="-12.7" x2="43.18" y2="-12.7" width="0.1524" layer="91"/>
+<pinref part="U$2" gate="G$1" pin="SCL"/>
+<wire x1="43.18" y1="-12.7" x2="35.56" y2="-12.7" width="0.1524" layer="91"/>
+<wire x1="-33.02" y1="-2.54" x2="-7.62" y2="-2.54" width="0.1524" layer="91"/>
+<wire x1="-7.62" y1="-2.54" x2="-7.62" y2="7.62" width="0.1524" layer="91"/>
+<wire x1="-7.62" y1="7.62" x2="43.18" y2="7.62" width="0.1524" layer="91"/>
+<wire x1="43.18" y1="7.62" x2="43.18" y2="-12.7" width="0.1524" layer="91"/>
+<junction x="43.18" y="-12.7"/>
 </segment>
 </net>
@@
 <pinref part="C4" gate="G$1" pin="-"/>
 <wire x1="5.08" y1="43.18" x2="5.08" y2="30.48" width="0.1524" layer="91"/>
-<pinref part="INPUT" gate="G$1" pin="PWR"/>
-<wire x1="5.08" y1="22.86" x2="5.08" y2="30.48" width="0.1524" layer="91"/>
 <junction x="5.08" y="30.48"/>
 <pinref part="C2" gate="G$1" pin="2"/>
@@
 <pinref part="GND2" gate="1" pin="GND"/>
 <junction x="73.66" y="-63.5"/>
+<pinref part="SW1" gate="G$1" pin="P$1"/>
+<wire x1="-40.64" y1="-53.34" x2="-50.8" y2="-53.34" width="0.1524" layer="91"/>
+<pinref part="S1" gate="G$1" pin="C"/>
+<wire x1="-50.8" y1="-53.34" x2="-50.8" y2="-33.02" width="0.1524" layer="91"/>
+<wire x1="-50.8" y1="-33.02" x2="-45.72" y2="-33.02" width="0.1524" layer="91"/>
+<wire x1="-50.8" y1="-53.34" x2="-50.8" y2="-68.58" width="0.1524" layer="91"/>
+<junction x="-50.8" y="-53.34"/>
+<wire x1="-50.8" y1="-68.58" x2="35.56" y2="-68.58" width="0.1524" layer="91"/>
+<wire x1="35.56" y1="-68.58" x2="35.56" y2="-63.5" width="0.1524" layer="91"/>
+<pinref part="U$2" gate="G$1" pin="GND"/>
+<wire x1="-33.02" y1="2.54" x2="-33.02" y2="30.48" width="0.1524" layer="91"/>
+<wire x1="-33.02" y1="30.48" x2="5.08" y2="30.48" width="0.1524" layer="91"/>
+</segment>
+<segment>
+<pinref part="AUDIO_INPUT" gate="G$1" pin="PWR"/>
+<pinref part="GND3" gate="1" pin="GND"/>
+<wire x1="-20.32" y1="68.58" x2="-20.32" y2="73.66" width="0.1524" layer="91"/>
 </segment>
 </net>
@@
 <junction x="50.8" y="-25.4"/>
 </segment>
+<segment>
+<pinref part="U$2" gate="G$1" pin="VCC"/>
+<pinref part="SUPPLY3" gate="G$1" pin="VCC"/>
+<wire x1="-33.02" y1="0" x2="-20.32" y2="0" width="0.1524" layer="91"/>
+</segment>
 </net>
 <net name="N$1" class="0">
 <segment>
-<pinref part="INPUT" gate="G$1" pin="GND"/>
+<pinref part="AUDIO_INPUT" gate="G$1" pin="GND"/>
 <pinref part="C3" gate="G$1" pin="1"/>
-<wire x1="5.08" y1="17.78" x2="10.16" y2="17.78" width="0.1524" layer="91"/>
-</segment>
-</net>
-<net name="N$6" class="0">
-<segment>
-<pinref part="R4" gate="G$1" pin="2"/>
-<pinref part="C3" gate="G$1" pin="2"/>
-<wire x1="20.32" y1="45.72" x2="17.78" y2="45.72" width="0.1524" layer="91"/>
-<wire x1="17.78" y1="45.72" x2="17.78" y2="17.78" width="0.1524" layer="91"/>
+<wire x1="-20.32" y1="63.5" x2="-15.24" y2="63.5" width="0.1524" layer="91"/>
 </segment>
 </net>
@@
 </segment>
 </net>
+<net name="N$10" class="0">
+<segment>
+<pinref part="M2" gate="G$1" pin="D2"/>
+<wire x1="0" y1="-30.48" x2="-25.4" y2="-30.48" width="0.1524" layer="91"/>
+<pinref part="S1" gate="G$1" pin="A"/>
+<wire x1="-25.4" y1="-30.48" x2="-25.4" y2="-25.4" width="0.1524" layer="91"/>
+</segment>
+</net>
+<net name="N$11" class="0">
+<segment>
+<pinref part="M2" gate="G$1" pin="D3"/>
+<wire x1="0" y1="-33.02" x2="-25.4" y2="-33.02" width="0.1524" layer="91"/>
+<pinref part="S1" gate="G$1" pin="B"/>
+<wire x1="-25.4" y1="-33.02" x2="-25.4" y2="-40.64" width="0.1524" layer="91"/>
+</segment>
+</net>
+<net name="N$12" class="0">
+<segment>
+<pinref part="M2" gate="G$1" pin="D4"/>
+<wire x1="0" y1="-35.56" x2="-20.32" y2="-35.56" width="0.1524" layer="91"/>
+<wire x1="-20.32" y1="-35.56" x2="-20.32" y2="-53.34" width="0.1524" layer="91"/>
+<pinref part="SW1" gate="G$1" pin="P$2"/>
+<wire x1="-20.32" y1="-53.34" x2="-30.48" y2="-53.34" width="0.1524" layer="91"/>
+</segment>
+</net>
+<net name="N$6" class="0">
+<segment>
+<pinref part="R4" gate="G$1" pin="2"/>
+<pinref part="C3" gate="G$1" pin="2"/>
+<wire x1="20.32" y1="45.72" x2="20.32" y2="63.5" width="0.1524" layer="91"/>
+<wire x1="20.32" y1="63.5" x2="-7.62" y2="63.5" width="0.1524" layer="91"/>
+</segment>
+</net>

Commit message: Shortwave receiver tester
Parts:
- renumbered S1 to RE
Other:
- note added: "Encoder"
- note added: "Step switch"
Changed lines of the file:
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@@
 <part name="GND2" library="supply1" library_urn="urn:adsk.eagle:library:371" deviceset="GND" device=""/>
 <part name="C5" library="rcl" library_urn="urn:adsk.eagle:library:334" deviceset="CX" device="XC10B6" package3d_urn="urn:adsk.eagle:package:23700/1" value="10nF"/>
-<part name="S1" library="SparkFun-Switches" library_urn="urn:adsk.eagle:library:535" deviceset="ENCODER" device="" package3d_urn="urn:adsk.eagle:package:40145/1"/>
+<part name="RE" library="SparkFun-Switches" library_urn="urn:adsk.eagle:library:535" deviceset="ENCODER" device="" package3d_urn="urn:adsk.eagle:package:40145/1"/>
 <part name="SW1" library="adafruit" library_urn="urn:adsk.eagle:library:420" deviceset="SWITCH_PUSHBUTTON" device="C&amp;K_KSS" package3d_urn="urn:adsk.eagle:package:6240958/1"/>
 <part name="SUPPLY3" library="supply2" library_urn="urn:adsk.eagle:library:372" deviceset="VCC" device="">
@@
 <sheet>
 <plain>
+<text x="-40.64" y="-58.42" size="1.778" layer="91">Step switch</text>
+<text x="-53.34" y="-27.94" size="1.778" layer="91">Encoder</text>
 </plain>
 <instances>
@@
 <attribute name="VALUE" x="85.344" y="23.241" size="1.778" layer="96"/>
 </instance>
-<instance part="S1" gate="G$1" x="-35.56" y="-33.02" smashed="yes">
+<instance part="RE" gate="G$1" x="-35.56" y="-33.02" smashed="yes">
 <attribute name="NAME" x="-40.64" y="-22.606" size="1.778" layer="95" font="vector"/>
 <attribute name="VALUE" x="-40.64" y="-43.434" size="1.778" layer="96" font="vector" align="top-left"/>
@@
 <pinref part="SW1" gate="G$1" pin="P$1"/>
 <wire x1="-40.64" y1="-53.34" x2="-50.8" y2="-53.34" width="0.1524" layer="91"/>
-<pinref part="S1" gate="G$1" pin="C"/>
+<pinref part="RE" gate="G$1" pin="C"/>
 <wire x1="-50.8" y1="-53.34" x2="-50.8" y2="-33.02" width="0.1524" layer="91"/>
 <wire x1="-50.8" y1="-33.02" x2="-45.72" y2="-33.02" width="0.1524" layer="91"/>
@@
 <pinref part="M2" gate="G$1" pin="D2"/>
 <wire x1="0" y1="-30.48" x2="-25.4" y2="-30.48" width="0.1524" layer="91"/>
-<pinref part="S1" gate="G$1" pin="A"/>
+<pinref part="RE" gate="G$1" pin="A"/>
 <wire x1="-25.4" y1="-30.48" x2="-25.4" y2="-25.4" width="0.1524" layer="91"/>
 </segment>
@@
 <pinref part="M2" gate="G$1" pin="D3"/>
 <wire x1="0" y1="-33.02" x2="-25.4" y2="-33.02" width="0.1524" layer="91"/>
-<pinref part="S1" gate="G$1" pin="B"/>
+<pinref part="RE" gate="G$1" pin="B"/>
 <wire x1="-25.4" y1="-33.02" x2="-25.4" y2="-40.64" width="0.1524" layer="91"/>
 </segment>
